File: PowerMeter2026-nRF/PowerMeter2026-nRF.kicad_sch (KiCad schematic)
At the start: 24 parts, among them J1 STRAIN, Q1 AO3401A, Q2 MMBT3906, SW1 CELL, U1 HT7733, U2 nRF52840 sense, U3 HX711

Commit message: Add files via upload
フットプリント設定完了。未配線。
Parts:
- BT1: footprint KUBTSS_parts:CellHolder_BH-311-1P24 -> KUBTSS:BatteryCell
- U2: footprint (none) -> KUBTSS:nRF52840 XIAO Sense
- U3: footprint Package_SO:SOP-16_3.9x9.9mm_P1.27mm -> Package_SO:JEITA_SOIC-16_3.9x9.9mm_P1.27mm
Connections:
- net +3V3: now also U2.3V3; no longer U2. (GND)
- net GND: now also U2.GND; no longer U2. (GND)
- no-connect marks 2 -> 10
Changed lines of the file:
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@@
 (kicad_sch
-	(version 20231120)
+	(version 20250114)
 	(generator "eeschema")
-	(generator_version "8.0")
+	(generator_version "9.0")
 	(paper "A4")
+	(text "Output Data with 80SPS"
+		(exclude_from_sim no)
+		(at 265.43 57.15 0)
+		(effects
+			(font
+				(size 1.27 1.27)
+			)
+		)
+	)
+	(text "D\n"
+		(exclude_from_sim no)
+		(at 180.086 109.474 0)
+		(effects
+			(font
+				(size 1.27 1.27)
+			)
+		)
+	)
+	(text "G"
+		(exclude_from_sim no)
+		(at 176.276 115.062 0)
+		(effects
+			(font
+				(size 1.27 1.27)
+			)
+		)
+	)
+	(text "HX711モジュールの素子の配置\n3.3V駆動"
+		(exclude_from_sim no)
+		(at 244.856 80.772 0)
+		(effects
+			(font
+				(size 1.27 1.27)
+			)
+		)
+	)
+	(text "S"
+		(exclude_from_sim no)
+		(at 169.672 106.934 0)
+		(effects
+			(font
+				(size 1.27 1.27)
+			)
+		)
+	)
+	(text "2~3Aクラスのインダクタを使う\n"
+		(exclude_from_sim no)
+		(at 76.708 33.782 0)
+		(effects
+			(font
+				(size 1.27 1.27)
+			)
+		)
+	)
+	(text "Use Internal Oscillator"
+		(exclude_from_sim no)
+		(at 265.176 61.976 0)
+		(effects
+			(font
+				(size 1.27 1.27)
+			)
+		)
+	)
+	(text "省電力のため"
+		(exclude_from_sim no)
+		(at 236.22 81.788 0)
+		(effects
+			(font
+				(size 1.27 1.27)
+			)
+		)
+	)
+	(text "L3のVinに可能な\n限り近づける"
+		(exclude_from_sim no)
+		(at 61.468 49.276 0)
+		(effects
+			(font
+				(size 1.27 1.27)
+			)
+		)
+	)
 	(junction
 		(at 252.73 54.61)
@@
 	)
 	(no_connect
+		(at 135.89 128.27)
+	)
+	(no_connect
+		(at 135.89 135.89)
+	)
+	(no_connect
 		(at 250.19 62.23)
 	)
 	(no_connect
+		(at 107.95 133.35)
+	)
+	(no_connect
 		(at 105.41 57.15)
 	)
+	(no_connect
+		(at 107.95 135.89)
+	)
+	(no_connect
+		(at 135.89 120.65)
+	)
+	(no_connect
+		(at 107.95 130.81)
+	)
+	(no_connect
+		(at 135.89 130.81)
+	)
+	(no_connect
+		(at 135.89 133.35)
+	)
 	(wire
 		(pts
@@
 	(wire
 		(pts
+			(xy 259.08 49.53) (xy 260.35 49.53)
+		)
+		(stroke
+			(width 0)
+			(type default)
+		)
+	)
+	(wire
+		(pts
 			(xy 252.73 54.61) (xy 250.19 54.61)
 		)
@@
 	(wire
 		(pts
-			(xy 190.5 60.96) (xy 190.5 59.69)
+			(xy 190.5 62.23) (xy 190.5 59.69)
 		)
 		(stroke
@@
 		)
 	)
-	(text "Output Data with 80SPS"
-		(exclude_from_sim no)
-		(at 265.43 57.15 0)
-		(effects
-			(font
-				(size 1.27 1.27)
-			)
-		)
-	)
-	(text "D\n"
-		(exclude_from_sim no)
-		(at 180.086 109.474 0)
-		(effects
-			(font
-				(size 1.27 1.27)
-			)
-		)
-	)
-	(text "G"
-		(exclude_from_sim no)
-		(at 176.276 115.062 0)
-		(effects
-			(font
-				(size 1.27 1.27)
-			)
-		)
-	)
-	(text "HX711モジュールの素子の配置\n3.3V駆動"
-		(exclude_from_sim no)
-		(at 244.856 80.772 0)
-		(effects
-			(font
-				(size 1.27 1.27)
-			)
-		)
-	)
-	(text "S"
-		(exclude_from_sim no)
-		(at 169.672 106.934 0)
-		(effects
-			(font
-				(size 1.27 1.27)
-			)
-		)
-	)
-	(text "2~3Aクラスのインダクタを使う\n"
-		(exclude_from_sim no)
-		(at 76.708 33.782 0)
-		(effects
-			(font
-				(size 1.27 1.27)
-			)
-		)
-	)
-	(text "Use Internal Oscillator"
-		(exclude_from_sim no)
-		(at 265.176 61.976 0)
-		(effects
-			(font
-				(size 1.27 1.27)
-			)
-		)
-	)
-	(text "省電力のため"
-		(exclude_from_sim no)
-		(at 236.22 81.788 0)
-		(effects
-			(font
-				(size 1.27 1.27)
-			)
-		)
-	)
-	(text "L3のVinに可能な\n限り近づける"
-		(exclude_from_sim no)
-		(at 61.468 49.276 0)
-		(effects
-			(font
-				(size 1.27 1.27)
-			)
-		)
-	)
 	(global_label "CLK"
 		(shape output)
@@
 			)
 		)
-		(property "Footprint" "KUBTSS_parts:CellHolder_BH-311-1P24"
+		(property "Footprint" "KUBTSS:BatteryCell"
 			(at 24.13 56.896 90)
 			(effects
@@
 			)
 		)
-		(property "Footprint" ""
+		(property "Footprint" "KUBTSS:nRF52840 XIAO Sense"
 			(at 120.65 130.81 0)
 			(effects
@@
 		(pin "P0.05"
 		)
-		(pin ""
+		(pin "VBUS"
 		)
-		(pin ""
+		(pin "3V3"
 		)
 		(pin "P0.02"
@@
 		(pin "P1.11"
 		)
-		(pin ""
+		(pin "GND"
 		)
 		(instances
@@
 	(symbol
 		(lib_id "power:GND")
-		(at 190.5 60.96 0)
+		(at 190.5 62.23 0)
 		(mirror y)
 		(unit 1)
@@
 		(dnp no)
 		(property "Reference" "#PWR011"
-			(at 190.5 67.31 0)
+			(at 190.5 68.58 0)
 			(effects
 				(font
@@
 		)
 		(property "Value" "GND"
-			(at 190.373 65.3542 0)
+			(at 190.373 66.6242 0)
 			(effects
 				(font
@@
 		)
 		(property "Footprint" ""
-			(at 190.5 60.96 0)
+			(at 190.5 62.23 0)
 			(effects
 				(font
@@
 		)
 		(property "Datasheet" ""
-			(at 190.5 60.96 0)
+			(at 190.5 62.23 0)
 			(effects
 				(font
@@
 		)
 		(property "Description" ""
-			(at 190.5 60.96 0)
+			(at 190.5 62.23 0)
 			(effects
 				(font
@@
 			)
 		)
-		(property "Footprint" "Package_SO:SOP-16_3.9x9.9mm_P1.27mm"
+		(property "Footprint" "Package_SO:JEITA_SOIC-16_3.9x9.9mm_P1.27mm"
 			(at 240.03 64.77 0)
 			(effects
@@
 	(symbol
 		(lib_id "power:GND")
-		(at 259.08 49.53 90)
+		(at 260.35 49.53 90)
 		(unit 1)
 		(exclude_from_sim no)
@@
 		(dnp no)
 		(property "Reference" "#PWR017"
-			(at 265.43 49.53 0)
+			(at 266.7 49.53 0)
 			(effects
 				(font
@@
 		)
 		(property "Value" "GND"
-			(at 262.3312 49.403 90)
+			(at 263.6012 49.403 90)
 			(effects
 				(font
@@
 		)
 		(property "Footprint" ""
-			(at 259.08 49.53 0)
+			(at 260.35 49.53 0)
 			(effects
 				(font
@@
 		)
 		(property "Datasheet" ""
-			(at 259.08 49.53 0)
+			(at 260.35 49.53 0)
 			(effects
 				(font
@@
 		)
 		(property "Description" ""
-			(at 259.08 49.53 0)
+			(at 260.35 49.53 0)
 			(effects
 				(font
@@
 		)
 	)
+	(embedded_fonts no)
 )

Commit message: Add files via upload
Parts:
- removed C3: 22u, Capacitor_SMD:C_1210_3225Metric, symbol Device:C
- removed L1: 47uH, Inductor_THT:L_Axial_L11.0mm_D4.5mm_P5.08mm_Vertical_Fastron_MECC, symbol Device:L
- removed U1: HT7733, Package_TO_SOT_SMD:SOT-23-5, symbol KUBTSS_parts:HT77xxA_CE_SOT25
- added C10, C11: 0.1u, Capacitor_SMD:C_0603_1608Metric, symbol Device:C_Small
- added C12, C9: 10u, Capacitor_SMD:C_0603_1608Metric, symbol Device:C_Small
- added J2: STRAIN_L, Connector_JST:JST_XH_S4B-XH-A_1x04_P2.50mm_Horizontal, symbol Connector:Conn_01x04_Male
- added J3, J4: USB_C_Receptacle_USB2.0_16P, Connector_USB:USB_C_Receptacle_HRO_TYPE-C-31-M-12, symbol Connector:USB_C_Receptacle_USB2.0_16P
- added Q3: MMBT3906, Package_TO_SOT_SMD:SOT-23, symbol Transistor_BJT:MMBT3906
- added R10: 10k, Resistor_SMD:R_0603_1608Metric, symbol Device:R_US
- added R11, R12, R13: 5.1k, Resistor_SMD:R_0603_1608Metric, symbol Device:R_US
- added R7, R8: 100, Resistor_SMD:R_0603_1608Metric, symbol Device:R_US
- added R9: 14k, Resistor_SMD:R_0603_1608Metric, symbol Device:R_US
- added U1: NCP1117-3.3_TO252, Package_TO_SOT_SMD:TO-252-2, symbol Regulator_Linear:NCP1117-3.3_TO252
- added U4: HX711_L, Package_SO:JEITA_SOIC-16_3.9x9.9mm_P1.27mm, symbol PowerMeter2023-rescue:HX711-RotationBoard_parts
- C1: value 47u -> 2.2u; footprint Capacitor_SMD:C_1210_3225Metric -> Capacitor_SMD:C_0603_1608Metric
- C2: value 0.1u -> 0.33u
- J1: value STRAIN -> STRAIN_R
- R1: value 100k -> 5.1k
- U3: value HX711 -> HX711_R
Connections:
- net +3V3: now also C1.1, C9.2, J2.1 (Pin_1), J3.A4 (VBUS), J3.A9 (VBUS), J3.B4 (VBUS), J3.B9 (VBUS), J4.A4 (VBUS), J4.A9 (VBUS), J4.B4 (VBUS), J4.B9 (VBUS), Q3.3 (C), R9.1, U1.2 (VO), U4.3 (AVDD); no longer C2.2, R1.2
- net +VDD: now also C12.2, Q3.2 (E), U4.1 (VSUP), U4.15 (RATE), U4.16 (DVDD)
- net ADC_BAT: now also U2.P1.11 (D6/TX), J3.A8 (SBU1), J4.A8 (SBU1); no longer U2.P0.29 (D3/A3)
- net GND: now also C2.2, R1.2, C10.2, C12.1, C9.1, J2.4 (Pin_4), J3.A1 (GND), J3.A12 (GND), J3.B1 (GND), J3.B12 (GND), J3.S1 (SHIELD), J4.A1 (GND), J4.A12 (GND), J4.B1 (GND), J4.B12 (GND), J4.S1 (SHIELD), R10.2, R11.1, R12.2, R13.1, U1.1 (GND), U4.10 (INPB), U4.14 (XI), U4.5 (AGND), U4.9 (INNB)
- net SW: now also U2.P1.14 (D9/MISO); no longer U2.P0.02 (D0/A0)
- net at BT1.1 (+): now also SW1.1 (A); no longer SW1.2 (B)
- net DAT_L: now reaches U2.P1.12 (D7/RX)
- net DAT_L: now also J3.A6 (D+), J4.A6 (D+), U4.12 (DOUT)
- net CLK_L: now reaches U2.P1.13 (D8/SCK)
- net CLK_L: now also J3.B6 (D+), J4.B6 (D+), U4.11 (PD_SCK)
- net at C2.1: now also D1.2 (A), SW1.2 (B), U1.3 (VI); no longer R1.1
- net CLK renamed CLK_R
- net CLK_R: now also U2.P0.29 (D3/A3), J3.A7 (D-), J4.A7 (D-); no longer U2.P0.28 (D2/A2)
- net DAT: no longer names the net of U2.P0.03 (D1/A1)
- net DAT: no longer U3.12 (DOUT)
- net INNA renamed INNA_R
- net INPA renamed INPA_R
- new net: C10.1, U4.6 (VBG)
- new net: R10.1, R9.2, U4.4 (VFB)
- new net: J3.A5 (CC1), R1.1
- new net: C11.1, R8.2, U4.8 (INPA)
- new net: C11.2, R7.2, U4.7 (INNA)
- new net: J4.A5 (CC1), R12.1
- new net: J4.B5 (CC2), R13.2
- new net: J3.B5 (CC2), R11.2
- new net: Q3.1 (B), U4.2 (BASE)
- new net DAT_R: J3.B7 (D-), J4.B7 (D-), U2.P0.28 (D2/A2), U3.12 (DOUT)
- new net INNA_L: J2.3 (Pin_3), R7.1
- new net INPA_L: J2.2 (Pin_2), R8.1
- no-connect marks 10 -> 11
Other:
- note added: "//2~3Aクラスのインダクタを使う"
- note added: "3.7V"
- note removed: "2~3Aクラスのインダクタを使う"
- note removed: "L3のVinに可能な 限り近づける"
- moved on the sheet: BT1, Q1, SW1, U2

Commit message: Add files via upload
Connections:
- net +3V3: now also D1.2 (A); no longer D1.1 (K)
- net at C2.1, SW1.2 (B), U1.3 (VI): now also D1.1 (K); no longer D1.2 (A)
Other:
- moved on the sheet: D1
Changed lines of the file:
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@@
 	(symbol
 		(lib_id "Device:D_Schottky")
-		(at 97.79 40.64 180)
+		(at 97.79 40.64 0)
 		(unit 1)
 		(exclude_from_sim no)
@@
 		(fields_autoplaced yes)
 		(property "Reference" "D1"
-			(at 98.1075 34.29 0)
+			(at 97.4725 34.29 0)
 			(effects
 				(font
@@
 		)
 		(property "Value" "RB160M"
-			(at 98.1075 36.83 0)
+			(at 97.4725 36.83 0)
 			(effects
 				(font

Commit message: Add files via upload
Parts:
- U1: value NCP1117-3.3_TO252 -> NJM2845DL1-33
Connections:
- net +3V3: now also C12.2, C8.2, Q2.2 (E), Q3.2 (E), U3.1 (VSUP), U3.15 (RATE), U3.16 (DVDD), U4.1 (VSUP), U4.15 (RATE), U4.16 (DVDD); no longer C5.2, C9.2, J1.1 (Pin_1), J2.1 (Pin_1), Q2.3 (C), Q3.3 (C), R5.1, R9.1, U3.3 (AVDD), U4.3 (AVDD)
- net +VDD: no longer C12.2, C8.2, Q2.2 (E), Q3.2 (E), U3.1 (VSUP), U3.15 (RATE), U3.16 (DVDD), U4.1 (VSUP), U4.15 (RATE), U4.16 (DVDD)
- new net +VDDA_L: C9.2, J2.1 (Pin_1), Q3.3 (C), R9.1, U4.3 (AVDD)
- new net +VDDA_R: C5.2, J1.1 (Pin_1), Q2.3 (C), R5.1, U3.3 (AVDD)
Changed lines of the file:
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@@
 	(text "//2~3Aクラスのインダクタを使う\n"
 		(exclude_from_sim no)
-		(at 76.962 8.89 0)
+		(at 78.232 26.67 0)
 		(effects
 			(font
@@
 			)
 		)
-		(property "Value" "+3V3"
+		(property "Value" "+VDDA_R"
 			(at 190.119 46.2788 90)
 			(effects
@@
 			)
 		)
-		(property "Value" "+3V3"
+		(property "Value" "+VDDA_R"
 			(at 208.8388 46.609 90)
 			(effects
@@
 			)
 		)
-		(property "Value" "NCP1117-3.3_TO252"
+		(property "Value" "NJM2845DL1-33"
 			(at 97.79 48.26 0)
 			(effects
@@
 			)
 		)
-		(property "Value" "+VDD"
+		(property "Value" "+3V3"
 			(at 241.3 110.49 0)
 			(effects
@@
 			)
 		)
-		(property "Value" "+3V3"
+		(property "Value" "+VDDA_L"
 			(at 178.689 114.8588 90)
 			(effects
@@
 			)
 		)
-		(property "Value" "+VDD"
+		(property "Value" "+3V3"
 			(at 252.73 41.91 0)
 			(effects
@@
 			)
 		)
-		(property "Value" "+3V3"
+		(property "Value" "+VDDA_L"
 			(at 197.4088 115.189 90)
 			(effects

Commit message: Add files via upload
Parts:
- removed BT1: Battery_Cell, KUBTSS:BatteryCell, symbol Device:Battery_Cell
- removed C1: 2.2u, Capacitor_SMD:C_0603_1608Metric, symbol Device:C
- removed C10, C11: 0.1u, Capacitor_SMD:C_0603_1608Metric, symbol Device:C_Small
- removed C12, C8, C9: 10u, Capacitor_SMD:C_0603_1608Metric, symbol Device:C_Small
- removed C2: 0.33u, Capacitor_SMD:C_0603_1608Metric, symbol Device:C
- removed C4: 0.1u, Capacitor_SMD:C_0603_1608Metric, symbol Device:C
- removed D1: RB160M, Diode_SMD:D_0603_1608Metric, symbol Device:D_Schottky
- removed J1: STRAIN_R, Connector_JST:JST_XH_S4B-XH-A_1x04_P2.50mm_Horizontal, symbol Connector:Conn_01x04_Male
- removed J2: STRAIN_L, Connector_JST:JST_XH_S4B-XH-A_1x04_P2.50mm_Horizontal, symbol Connector:Conn_01x04_Male
- removed J3, J4: USB_C_Receptacle_USB2.0_16P, Connector_USB:USB_C_Receptacle_HRO_TYPE-C-31-M-12, symbol Connector:USB_C_Receptacle_USB2.0_16P
- removed Q2, Q3: MMBT3906, Package_TO_SOT_SMD:SOT-23, symbol Transistor_BJT:MMBT3906
- removed R1, R13: 5.1k, Resistor_SMD:R_0603_1608Metric, symbol Device:R_US
- removed R10, R6: 10k, Resistor_SMD:R_0603_1608Metric, symbol Device:R_US
- removed R2: 1k, Resistor_SMD:R_0603_1608Metric, symbol Device:R_US
- removed R7, R8: 100, Resistor_SMD:R_0603_1608Metric, symbol Device:R_US
- removed R9: 14k, Resistor_SMD:R_0603_1608Metric, symbol Device:R_US
- removed SW1: CELL, KUBTSS:toggle, symbol Switch:SW_SPDT
- removed U1: NJM2845DL1-33, Package_TO_SOT_SMD:TO-252-2, symbol Regulator_Linear:NCP1117-3.3_TO252
- removed U3: HX711_R, Package_SO:JEITA_SOIC-16_3.9x9.9mm_P1.27mm, symbol PowerMeter2023-rescue:HX711-RotationBoard_parts
- removed U4: HX711_L, Package_SO:JEITA_SOIC-16_3.9x9.9mm_P1.27mm, symbol PowerMeter2023-rescue:HX711-RotationBoard_parts
- added BT2: Battery_Cell, KUBTSS:BatteryCell, symbol Device:Battery_Cell
- added C13, C15: 1u, Capacitor_SMD:C_0603_1608Metric, symbol Device:C_Small
- added C14: 220u, Capacitor_SMD:C_0603_1608Metric, symbol Device:C_Small
- added C4: 0.1u, Capacitor_SMD:C_0603_1608Metric, symbol Device:C_Small
- added C8: 0.1u, Capacitor_SMD:C_0603_1608Metric, symbol Device:C
- added D6: RB160M, Diode_SMD:D_SOD-123, symbol Device:D_Schottky
- added J3, J4: Conn_01x10_Pin, Connector_PinHeader_2.54mm:PinHeader_2x05_P2.54mm_Horizontal, symbol Connector:Conn_01x10_Pin
- added J5: STRAIN_R, Connector_PinHeader_2.54mm:PinHeader_1x04_P2.54mm_Vertical, symbol Connector:Conn_01x04_Male
- added SW2: CELL, KUBTSS:toggle, symbol Switch:SW_SPDT
- added U3: TPS76133SF5, Package_TO_SOT_SMD:SOT-23-5, symbol Regulator_Linear:TPS76901
- added U5: ADS131M02, Package_SO:TSSOP-20_4.4x6.5mm_P0.65mm, symbol KUBTSS:ADS131M02
- C5: value 10u -> 1u
- C6, C7: value 0.1u -> 1u
- R11, R12: value 5.1k -> 100
- R3: value 100 -> 22k
- R4: value 100 -> 100k
- R5: value 14k -> 100k
Connections:
- net DAT_R is gone; now on net SW: U2.P0.28 (D2/A2)
- net INNA_R is gone; now on an unnamed net: R3.1
- net INPA_R is gone; now on net ADC_BAT: R4.1
- net +3V3: now also C7.1, C13.2, C15.2, D6.2 (A), J3.1 (Pin_1), J4.1 (Pin_1), U3.5 (OUT), U5.1 (AVDD), U5.11 (SYNC/RST), U5.20 (DVDD)
- net +VDD: now also J5.1 (Pin_1), U5.6 (AIN1P)
- net ADC_BAT: now also R5.1, C8.1, J3.8 (Pin_8), J4.8 (Pin_8)
- net GND: now also C5.2, C7.2, R5.2, BT2.2 (-), C13.1, C14.1, C15.1, C8.2, J3.10 (Pin_10), J4.10 (Pin_10), J5.4 (Pin_4), U3.2 (GND), U5.19 (DGND), U5.2 (AGND), U5.5 (AIN1N); no longer C5.1, R11.1, R12.2
- net SW: now also J3.9 (Pin_9), J4.9 (Pin_9); no longer U2.P1.14 (D9/MISO)
- net INNA: now reaches R12.1
- net INNA: now also J5.3 (Pin_3)
- net at R11.2: now also C4.2, U5.3 (AIN0P)
- net CLK: now reaches U2.P0.02 (D0/A0)
- net CLK: now also J3.2 (Pin_2), J4.2 (Pin_2), U5.17 (CLKIN)
- net DRDY: now reaches U2.P0.03 (D1/A1)
- net DRDY: now also J3.6 (Pin_6), J4.6 (Pin_6), U5.13 (DRDY)
- net MOSI: now reaches U2.P1.15 (D10/MOSI)
- net MOSI: now also J3.3 (Pin_3), J4.3 (Pin_3), U5.16 (DIN)
- net at R4.2: now also C6.1, D6.1 (K), SW2.2 (B), U3.1 (IN); no longer C7.1
- net at R3.2: now also C5.1, U3.3 (~{EN}); no longer C7.2
- removed net +VDDA_R: C5.2, R5.1
- net CLK_L renamed SCK
- net SCK: now also J3.5 (Pin_5), J4.5 (Pin_5), U5.14 (SCLK)
- net CLK_R: no longer names the net of U2.P0.29 (D3/A3)
- net DAT_L renamed CS
- net CS: now also J3.7 (Pin_7), J4.7 (Pin_7), U5.12 (CS)
- new net: BT2.1 (+), SW2.1 (A)
- new net: C4.1, R12.2, U5.4 (AIN0N)
- new net: C14.2, U5.18 (CAP)
- new net INPA: J5.2 (Pin_2), R11.1
- new net MISO: J3.4 (Pin_4), J4.4 (Pin_4), U2.P1.14 (D9/MISO), U5.15 (DOUT)
- no-connect marks 11 -> 10
Other:
- note added: "AGNDとDGNDはデバイスの近くで一点接続することが推奨されている"
- note added: "max:150mA"
- note added: "ひずみゲージ"
- note added: "スライドスイッチ"
- note removed: "//2~3Aクラスのインダクタを使う"
- note removed: "HX711モジュールの素子の配置 3.3V駆動"
- note removed: "Output Data with 80SPS"
- note removed: "Use Internal Oscillator"
- note removed: "省電力のため"
- moved on the sheet: Q1, U2

Commit message: Add files via upload
Parts:
- J3, J4: value Conn_01x10_Pin -> Conn_JST_PHD_S10B_PHDSS; footprint Connector_PinHeader_2.54mm:PinHeader_2x05_P2.54mm_Horizontal -> Connector_JST:JST_PHD_S10B-PHDSS_2x05_P2.00mm_Horizontal
Other:
- moved on the sheet: J4
Changed lines of the file:
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@@
 	(wire
 		(pts
-			(xy 157.48 152.4) (xy 168.91 152.4)
+			(xy 161.29 152.4) (xy 172.72 152.4)
 		)
 		(stroke
@@
 	(wire
 		(pts
-			(xy 167.64 147.32) (xy 157.48 147.32)
+			(xy 171.45 147.32) (xy 161.29 147.32)
 		)
 		(stroke
@@
 	(wire
 		(pts
-			(xy 167.64 149.86) (xy 157.48 149.86)
+			(xy 171.45 149.86) (xy 161.29 149.86)
 		)
 		(stroke
@@
 	(wire
 		(pts
-			(xy 157.48 157.48) (xy 168.91 157.48)
+			(xy 161.29 157.48) (xy 172.72 157.48)
 		)
 		(stroke
@@
 	(wire
 		(pts
-			(xy 167.64 142.24) (xy 157.48 142.24)
+			(xy 171.45 142.24) (xy 161.29 142.24)
 		)
 		(stroke
@@
 	(wire
 		(pts
-			(xy 168.91 157.48) (xy 168.91 162.56)
+			(xy 172.72 157.48) (xy 172.72 162.56)
 		)
 		(stroke
@@
 	(wire
 		(pts
-			(xy 165.1 154.94) (xy 157.48 154.94)
+			(xy 168.91 154.94) (xy 161.29 154.94)
 		)
 		(stroke
@@
 	(wire
 		(pts
-			(xy 167.64 137.16) (xy 157.48 137.16)
+			(xy 171.45 137.16) (xy 161.29 137.16)
 		)
 		(stroke
@@
 	(wire
 		(pts
-			(xy 167.64 139.7) (xy 157.48 139.7)
+			(xy 171.45 139.7) (xy 161.29 139.7)
 		)
 		(stroke
@@
 	(wire
 		(pts
-			(xy 167.64 144.78) (xy 157.48 144.78)
+			(xy 171.45 144.78) (xy 161.29 144.78)
 		)
 		(stroke
@@
 	(wire
 		(pts
-			(xy 157.48 134.62) (xy 182.88 134.62)
+			(xy 161.29 134.62) (xy 186.69 134.62)
 		)
 		(stroke
@@
 	(wire
 		(pts
-			(xy 182.88 132.08) (xy 182.88 134.62)
+			(xy 186.69 132.08) (xy 186.69 134.62)
 		)
 		(stroke
@@
 	(global_label "SW"
 		(shape output)
-		(at 165.1 154.94 0)
+		(at 168.91 154.94 0)
 		(fields_autoplaced yes)
 		(effects
@@
 		)
 		(property "Intersheetrefs" "${INTERSHEET_REFS}"
-			(at 170.7461 154.94 0)
+			(at 174.5561 154.94 0)
 			(effects
 				(font
@@
 	(global_label "MOSI"
 		(shape input)
-		(at 167.64 139.7 0)
+		(at 171.45 139.7 0)
 		(fields_autoplaced yes)
 		(effects
@@
 		)
 		(property "Intersheetrefs" "${INTERSHEET_REFS}"
-			(at 175.2214 139.7 0)
+			(at 179.0314 139.7 0)
 			(effects
 				(font
@@
 	(global_label "DRDY"
 		(shape output)
-		(at 167.64 147.32 0)
+		(at 171.45 147.32 0)
 		(fields_autoplaced yes)
 		(effects
@@
 		)
 		(property "Intersheetrefs" "${INTERSHEET_REFS}"
-			(at 175.5238 147.32 0)
+			(at 179.3338 147.32 0)
 			(effects
 				(font
@@
 	(global_label "ADC_BAT"
 		(shape input)
-		(at 168.91 152.4 0)
+		(at 172.72 152.4 0)
 		(fields_autoplaced yes)
 		(effects
@@
 		)
 		(property "Intersheetrefs" "${INTERSHEET_REFS}"
-			(at 179.8176 152.4 0)
+			(at 183.6276 152.4 0)
 			(effects
 				(font
@@
 	(global_label "SCK"
 		(shape output)
-		(at 167.64 144.78 0)
+		(at 171.45 144.78 0)
 		(fields_autoplaced yes)
 		(effects
@@
 		)
 		(property "Intersheetrefs" "${INTERSHEET_REFS}"
-			(at 174.3747 144.78 0)
+			(at 178.1847 144.78 0)
 			(effects
 				(font
@@
 	(global_label "CS"
 		(shape output)
-		(at 167.64 149.86 0)
+		(at 171.45 149.86 0)
 		(fields_autoplaced yes)
 		(effects
@@
 		)
 		(property "Intersheetrefs" "${INTERSHEET_REFS}"
-			(at 173.1047 149.86 0)
+			(at 176.9147 149.86 0)
 			(effects
 				(font
@@
 	(global_label "CLK"
 		(shape input)
-		(at 167.64 137.16 0)
+		(at 171.45 137.16 0)
 		(fields_autoplaced yes)
 		(effects
@@
 		)
 		(property "Intersheetrefs" "${INTERSHEET_REFS}"
-			(at 174.1933 137.16 0)
+			(at 178.0033 137.16 0)
 			(effects
 				(font
@@
 	(global_label "MISO"
 		(shape output)
-		(at 167.64 142.24 0)
+		(at 171.45 142.24 0)
 		(fields_autoplaced yes)
 		(effects
@@
 		)
 		(property "Intersheetrefs" "${INTERSHEET_REFS}"
-			(at 175.2214 142.24 0)
+			(at 179.0314 142.24 0)
 			(effects
 				(font
@@
 			)
 		)
-		(property "Value" "Conn_01x10_Pin"
+		(property "Value" "Conn_JST_PHD_S10B_PHDSS"
 			(at 109.855 130.81 0)
 			(effects
@@
 			)
 		)
-		(property "Footprint" "Connector_PinHeader_2.54mm:PinHeader_2x05_P2.54mm_Horizontal"
+		(property "Footprint" "Connector_JST:JST_PHD_S10B-PHDSS_2x05_P2.00mm_Horizontal"
 			(at 109.22 143.51 0)
 			(effects
@@
 	(symbol
 		(lib_id "power:GND")
-		(at 168.91 162.56 0)
+		(at 172.72 162.56 0)
 		(unit 1)
 		(exclude_from_sim no)
@@
 		(fields_autoplaced yes)
 		(property "Reference" "#PWR027"
-			(at 168.91 168.91 0)
+			(at 172.72 168.91 0)
 			(effects
 				(font
@@
 		)
 		(property "Value" "GND"
-			(at 168.91 167.64 0)
+			(at 172.72 167.64 0)
 			(effects
 				(font
@@
 		)
 		(property "Footprint" ""
-			(at 168.91 162.56 0)
+			(at 172.72 162.56 0)
 			(effects
 				(font
@@
 		)
 		(property "Datasheet" ""
-			(at 168.91 162.56 0)
+			(at 172.72 162.56 0)
 			(effects
 				(font
@@
 		)
 		(property "Description" "Power symbol creates a global label with name \"GND\" , ground"
-			(at 168.91 162.56 0)
+			(at 172.72 162.56 0)
 			(effects
 				(font
@@
 	(symbol
 		(lib_id "power:+3V3")
-		(at 182.88 132.08 0)
+		(at 186.69 132.08 0)
 		(unit 1)
 		(exclude_from_sim no)
@@
 		(fields_autoplaced yes)
 		(property "Reference" "#PWR028"
-			(at 182.88 135.89 0)
+			(at 186.69 135.89 0)
 			(effects
 				(font
@@
 		)
 		(property "Value" "+3V3"
-			(at 182.88 127 0)
+			(at 186.69 127 0)
 			(effects
 				(font
@@
 		)
 		(property "Footprint" ""
-			(at 182.88 132.08 0)
+			(at 186.69 132.08 0)
 			(effects
 				(font
@@
 		)
 		(property "Datasheet" ""
-			(at 182.88 132.08 0)
+			(at 186.69 132.08 0)
 			(effects
 				(font
@@
 		)
 		(property "Description" "Power symbol creates a global label with name \"+3V3\""
-			(at 182.88 132.08 0)
+			(at 186.69 132.08 0)
 			(effects
 				(font
@@
 	(symbol
 		(lib_id "Connector:Conn_01x10_Pin")
-		(at 152.4 144.78 0)
+		(at 156.21 144.78 0)
 		(unit 1)
 		(exclude_from_sim no)
@@
 		(fields_autoplaced yes)
 		(property "Reference" "J4"
-			(at 153.035 129.54 0)
+			(at 156.845 129.54 0)
 			(effects
 				(font
@@
 			)
 		)
-		(property "Value" "Conn_01x10_Pin"
-			(at 153.035 132.08 0)
+		(property "Value" "Conn_JST_PHD_S10B_PHDSS"
+			(at 156.845 132.08 0)
 			(effects
 				(font
@@
 			)
 		)
-		(property "Footprint" "Connector_PinHeader_2.54mm:PinHeader_2x05_P2.54mm_Horizontal"
-			(at 152.4 144.78 0)
+		(property "Footprint" "Connector_JST:JST_PHD_S10B-PHDSS_2x05_P2.00mm_Horizontal"
+			(at 156.21 144.78 0)
 			(effects
 				(font
@@
 		)
 		(property "Datasheet" "~"
-			(at 152.4 144.78 0)
+			(at 156.21 144.78 0)
 			(effects
 				(font
@@
 		)
 		(property "Description" "Generic connector, single row, 01x10, script generated"
-			(at 152.4 144.78 0)
+			(at 156.21 144.78 0)
 			(effects
 				(font
