File: PowerMeter2026-nRF/PowerMeter2026-nRF.kicad_sch (KiCad schematic)
At the start: 23 parts, among them J3 Conn_JST_PHD_S10B_PHDSS, J4 Conn_JST_PHD_S10B_PHDSS, J5 STRAIN_R, Q1 AO3401A, SW2 CELL, U2 nRF52840 sense, U3 TPS76133SF5, U5 ADS131M02

Commit message: Add files via upload
配線完了。基板設計完了。
Connections:
- net +3V3: now also J3.10 (Pin_10); no longer J3.1 (Pin_1), J4.1 (Pin_1), U2.3V3
- net ADC_BAT: no longer J4.8 (Pin_8), U2.P1.11 (D6/TX)
- net CLK: now also J3.7 (Pin_7); no longer J3.2 (Pin_2), J4.2 (Pin_2), U2.P0.02 (D0/A0)
- net CS: now also J3.4 (Pin_4); no longer J3.7 (Pin_7), J4.7 (Pin_7), U2.P1.12 (D7/RX)
- net DRDY: now also J3.2 (Pin_2); no longer J3.6 (Pin_6), J4.6 (Pin_6), U2.P0.03 (D1/A1)
- net GND: now also J3.6 (Pin_6); no longer J3.10 (Pin_10), J4.10 (Pin_10), U2.GND
- net MISO: now also J3.3 (Pin_3); no longer J3.4 (Pin_4), J4.4 (Pin_4), U2.P1.14 (D9/MISO)
- net MOSI: now also J3.5 (Pin_5); no longer J3.3 (Pin_3), J4.3 (Pin_3), U2.P1.15 (D10/MOSI)
- net SCK: now also J3.1 (Pin_1); no longer J3.5 (Pin_5), J4.5 (Pin_5), U2.P1.13 (D8/SCK)
- net SW: no longer J4.9 (Pin_9), U2.P0.28 (D2/A2)
- new net +3V3_M: J4.2 (Pin_2), U2.3V3
- new net ADC_BAT_M: J4.4 (Pin_4), U2.P1.11 (D6/TX)
- new net CLK_M: J4.3 (Pin_3), U2.P0.02 (D0/A0)
- new net CS_M: J4.8 (Pin_8), U2.P1.12 (D7/RX)
- new net DRDY_M: J4.10 (Pin_10), U2.P0.03 (D1/A1)
- new net GND_M: J4.6 (Pin_6), U2.GND
- new net MISO_M: J4.7 (Pin_7), U2.P1.14 (D9/MISO)
- new net MOSI_M: J4.5 (Pin_5), U2.P1.15 (D10/MOSI)
- new net SCK_M: J4.9 (Pin_9), U2.P1.13 (D8/SCK)
- new net SW_M: J4.1 (Pin_1), U2.P0.28 (D2/A2)
Other:
- moved on the sheet: J4
