File: PowerMeter2026-nRF/PowerMeter2026-nRF.kicad_pcb (KiCad board)
At the start: 2 copper layers, 24 parts, among them J1 STRAIN, Q1 AO3401A, Q2 MMBT3906, SW1 CELL, U1 HT7733, U2 nRF52840 sense, U3 HX711

Commit message: Add files via upload
Parts:
- removed C3: 22u, Capacitor_SMD:C_1210_3225Metric
- removed L1: 47uH, Inductor_THT:L_Axial_L11.0mm_D4.5mm_P5.08mm_Vertical_Fastron_MECC
- added C10: 0.1u, Capacitor_SMD:C_0603_1608Metric, B.Cu at (207.7, 42.4)
- added C11: 0.1u, Capacitor_SMD:C_0603_1608Metric, B.Cu at (207.7, 39.9)
- added C12: 10u, Capacitor_SMD:C_0603_1608Metric, B.Cu at (207.7, 37.4)
- added C9: 10u, Capacitor_SMD:C_0603_1608Metric, B.Cu at (207.7, 45.0)
- added J2: STRAIN_L, Connector_JST:JST_XH_S4B-XH-A_1x04_P2.50mm_Horizontal, F.Cu at (146.2, 37.7)
- added J3: USB_C_Receptacle_USB2.0_16P, Connector_USB:USB_C_Receptacle_HRO_TYPE-C-31-M-12, F.Cu at (170.2, 41.9)
- added J4: USB_C_Receptacle_USB2.0_16P, Connector_USB:USB_C_Receptacle_HRO_TYPE-C-31-M-12, B.Cu at (141.9, 57.9)
- added Q3: MMBT3906, Package_TO_SOT_SMD:SOT-23, B.Cu at (150.2, 44.7)
- added R10: 10k, Resistor_SMD:R_0603_1608Metric, B.Cu at (198.4, 45.9)
- added R11: 5.1k, Resistor_SMD:R_0603_1608Metric, B.Cu at (170.1, 39.7)
- added R12: 5.1k, Resistor_SMD:R_0603_1608Metric, F.Cu at (142.8, 64.4)
- added R13: 5.1k, Resistor_SMD:R_0603_1608Metric, F.Cu at (138.2, 64.2)
- added R7: 100, Resistor_SMD:R_0603_1608Metric, B.Cu at (211.7, 34.9)
- added R8: 100, Resistor_SMD:R_0603_1608Metric, B.Cu at (215.7, 47.5)
- added R9: 14k, Resistor_SMD:R_0603_1608Metric, B.Cu at (194.5, 44.6)
- added U4: HX711_L, Package_SO:JEITA_SOIC-16_3.9x9.9mm_P1.27mm, B.Cu at (156.2, 41.5)
- C1: value 47u -> 2.2u; footprint Capacitor_SMD:C_1210_3225Metric -> Capacitor_SMD:C_0603_1608Metric; moved to B.Cu
- C2: value 0.1u -> 0.33u; moved to B.Cu
- C4, C5, C6, C7, C8, Q1, Q2, R2, R3, R4, R5, R6, SW1: moved to B.Cu
- J1: value STRAIN -> STRAIN_R
- R1: value 100k -> 5.1k; moved to B.Cu
- U1: value HT7733 -> NCP1117-3.3_TO252; footprint Package_TO_SOT_SMD:SOT-23-5 -> Package_TO_SOT_SMD:TO-252-2
- U3: value HX711 -> HX711_R; moved to B.Cu
- moved J1 187.6 mm to (243.2, 44.7), turned to 90 degrees
- moved U3 176.5 mm to (231.8, 41.5)
- moved BT1 160.6 mm to (214.8, 41.0)
- moved Q2 152.4 mm to (225.8, 45.0), turned to 180 degrees
- moved R2 139.2 mm to (211.7, 47.5)
- moved C6 135.8 mm to (203.7, 37.4)
- moved R6 135.8 mm to (211.7, 37.4)
- moved C5 135.4 mm to (203.7, 39.9)
- moved R5 135.4 mm to (211.7, 39.9)
- moved C4 135.2 mm to (203.7, 42.4)
- moved R4 135.2 mm to (211.7, 42.4)
- moved C2 135.2 mm to (203.7, 45.0)
- moved C8 135.2 mm to (207.7, 47.5)
- moved R3 135.2 mm to (211.7, 45.0)
- moved D1 134.9 mm to (185.9, 39.9)
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Connections:
- net INNA renamed INNA_R
- net INPA renamed INPA_R
- C1 pad 1: Net-(SW1-A) -> +3V3
- C2 pad 1: Net-(U1-CE) -> Net-(D1-A)
- C2 pad 2: +3V3 -> GND
- R1 pad 1: Net-(U1-CE) -> Net-(J3-CC1)
- R1 pad 2: +3V3 -> GND
- SW1 pad 1: Net-(SW1-A) -> Net-(BT1-+)
- SW1 pad 2: Net-(BT1-+) -> Net-(D1-A)
- U1 pad 1: Net-(U1-CE) -> GND
- U1 pad 3: unconnected-(U1-NC-Pad3) -> Net-(D1-A)
- U2 pad P0.02: SW -> unconnected-(U2-D0/A0-PadP0.02)_1
- U2 pad P0.03: DAT -> unconnected-(U2-D1/A1-PadP0.03)_1
- U2 pad P0.28: CLK -> DAT_R
- U2 pad P0.29: ADC_BAT -> CLK_R
- U2 pad P1.11: unconnected-(U2-D6/TX-PadP1.11)_1 -> ADC_BAT
- U2 pad P1.12: unconnected-(U2-D7/RX-PadP1.12)_1 -> DAT_L
- U2 pad P1.13: unconnected-(U2-D8/SCK-PadP1.13)_1 -> CLK_L
- U2 pad P1.14: unconnected-(U2-D9/MISO-PadP1.14) -> SW
- U3 pad 11: CLK -> CLK_R
- U3 pad 12: DAT -> DAT_R

Commit message: Add files via upload
Parts:
- removed BT1: Battery_Cell, KUBTSS:BatteryCell
- removed C1: 2.2u, Capacitor_SMD:C_0603_1608Metric
- removed C10, C11: 0.1u, Capacitor_SMD:C_0603_1608Metric
- removed C12, C9: 10u, Capacitor_SMD:C_0603_1608Metric
- removed C2: 0.33u, Capacitor_SMD:C_0603_1608Metric
- removed D1: RB160M, Diode_SMD:D_0603_1608Metric
- removed J1: STRAIN_R, Connector_JST:JST_XH_S4B-XH-A_1x04_P2.50mm_Horizontal
- removed J2: STRAIN_L, Connector_JST:JST_XH_S4B-XH-A_1x04_P2.50mm_Horizontal
- removed Q2, Q3: MMBT3906, Package_TO_SOT_SMD:SOT-23
- removed R1, R13: 5.1k, Resistor_SMD:R_0603_1608Metric
- removed R10, R6: 10k, Resistor_SMD:R_0603_1608Metric
- removed R2: 1k, Resistor_SMD:R_0603_1608Metric
- removed R7, R8: 100, Resistor_SMD:R_0603_1608Metric
- removed R9: 14k, Resistor_SMD:R_0603_1608Metric
- removed SW1: CELL, KUBTSS:toggle
- removed U1: NCP1117-3.3_TO252, Package_TO_SOT_SMD:TO-252-2
- removed U4: HX711_L, Package_SO:JEITA_SOIC-16_3.9x9.9mm_P1.27mm
- added BT2: Battery_Cell, KUBTSS:BatteryCell, F.Cu at (222.6, 41.0)
- added C13: 1u, Capacitor_SMD:C_0603_1608Metric, B.Cu at (208.3, 43.8)
- added C14: 220u, Capacitor_SMD:C_0603_1608Metric, B.Cu at (217.7, 41.1)
- added C15: 1u, Capacitor_SMD:C_0603_1608Metric, B.Cu at (216.4, 43.7)
- added D6: RB160M, Diode_SMD:D_SOD-123, B.Cu at (238.6, 40.3)
- added J5: STRAIN_R, Connector_PinHeader_2.54mm:PinHeader_1x04_P2.54mm_Vertical, F.Cu at (194.2, 37.1)
- added SW2: CELL, KUBTSS:toggle, F.Cu at (250.6, 40.9)
- added U5: ADS131M02, Package_SO:TSSOP-20_4.4x6.5mm_P0.65mm, B.Cu at (212.3, 39.6)
- C5: value 10u -> 1u
- C6, C7: value 0.1u -> 1u
- C8: value 10u -> 0.1u
- J3: value USB_C_Receptacle_USB2.0_16P -> Conn_01x10_Pin; footprint Connector_USB:USB_C_Receptacle_HRO_TYPE-C-31-M-12 -> Connector_PinHeader_2.54mm:PinHeader_2x05_P2.54mm_Horizontal
- J4: value USB_C_Receptacle_USB2.0_16P -> Conn_01x10_Pin; footprint Connector_USB:USB_C_Receptacle_HRO_TYPE-C-31-M-12 -> Connector_PinHeader_2.54mm:PinHeader_2x05_P2.54mm_Horizontal; moved to F.Cu
- R11: value 5.1k -> 100
- R12: value 5.1k -> 100; moved to B.Cu
- R3: value 100 -> 22k
- R4: value 100 -> 100k
- R5: value 14k -> 100k
- U3: value HX711_R -> TPS76133SF5; footprint Package_SO:JEITA_SOIC-16_3.9x9.9mm_P1.27mm -> Package_TO_SOT_SMD:SOT-23-5
- moved R12 66.1 mm to (204.3, 40.1)
- moved Q1 63.0 mm to (203.8, 45.3), turned to -90 degrees
- moved C6 38.5 mm to (241.8, 43.2), turned to -90 degrees
- moved C5 36.3 mm to (239.5, 45.7), turned to 180 degrees
- moved R11 34.3 mm to (204.3, 41.7), turned to 180 degrees
- moved C7 33.7 mm to (236.0, 44.7), turned to -90 degrees
- moved R3 31.7 mm to (243.3, 43.2), turned to -90 degrees
- moved C8 26.7 mm to (233.4, 40.4)
- moved R4 22.0 mm to (233.4, 38.9)
- moved R5 21.8 mm to (233.4, 42.1)
- moved J3 19.9 mm to (189.7, 46.0), turned to 180 degrees
- moved U2 12.4 mm to (140.3, 78.2)
- moved J4 9.32 mm to (135.5, 64.7), turned to 90 degrees
- moved U3 7.34 mm to (238.9, 43.2), turned to 180 degrees
- moved C4 3.24 mm to (206.6, 40.9), turned to -90 degrees
Connections:
- C4 pad 1: ADC_BAT -> Net-(U5-AIN0N)
- C4 pad 2: GND -> Net-(U5-AIN0P)
- C5 pad 1: GND -> Net-(U3-~{EN})
- C5 pad 2: +3V3 -> GND
- C6 pad 1: Net-(U3-VBG) -> Net-(D6-K)
- C7 pad 1: Net-(U3-INPA) -> +3V3
- C7 pad 2: Net-(U3-INNA) -> GND
- C8 pad 1: GND -> ADC_BAT
- C8 pad 2: +VDD -> GND
- R11 pad 1: GND -> INPA
- R11 pad 2: Net-(J3-CC2) -> Net-(U5-AIN0P)
- R12 pad 1: Net-(J4-CC1) -> INNA
- R12 pad 2: GND -> Net-(U5-AIN0N)
- R3 pad 1: INNA_R -> Net-(D6-K)
- R3 pad 2: Net-(U3-INNA) -> Net-(U3-~{EN})
- R4 pad 1: INPA_R -> ADC_BAT
- R4 pad 2: Net-(U3-INPA) -> Net-(D6-K)
- R5 pad 1: +3V3 -> ADC_BAT
- R5 pad 2: Net-(U3-VFB) -> GND
- U2 pad P0.02: unconnected-(U2-D0/A0-PadP0.02)_1 -> CLK
- U2 pad P0.03: unconnected-(U2-D1/A1-PadP0.03)_1 -> DRDY
- U2 pad P0.28: DAT_R -> SW
- U2 pad P0.29: CLK_R -> unconnected-(U2-D3/A3-PadP0.29)_1
- U2 pad P1.12: DAT_L -> CS
- U2 pad P1.13: CLK_L -> SCK
- U2 pad P1.14: SW -> MISO
- U2 pad P1.15: unconnected-(U2-D10/MOSI-PadP1.15)_1 -> MOSI
- U3 pad 1: +VDD -> Net-(D6-K)
- U3 pad 2: Net-(Q2-B) -> GND
- U3 pad 3: +3V3 -> Net-(U3-~{EN})
- U3 pad 4: Net-(U3-VFB) -> unconnected-(U3-NC-Pad4)
- U3 pad 5: GND -> +3V3
Other:
- board text added: "20×32"
- board text added: "72×15"

Commit message: Add files via upload
Parts:
- J3, J4: footprint Connector_PinHeader_2.54mm:PinHeader_2x05_P2.54mm_Horizontal -> Connector_JST:JST_PHD_S10B-PHDSS_2x05_P2.00mm_Horizontal
- moved J4 9.68 mm to (144.9, 67.0), turned to 180 degrees
- moved J3 9.20 mm to (191.6, 37.0), turned to -90 degrees
- moved J5 0.59 mm to (194.8, 37.0)
- moved U2 0.24 mm to (140.4, 78.5)

Commit message: Add files via upload
配線完了。基板設計完了。
Parts:
- J3, J4: value Conn_01x10_Pin -> Conn_JST_PHD_S10B_PHDSS
- moved J4 31.9 mm to (176.8, 66.5)
- moved U2 31.7 mm to (172.1, 77.8)
- moved J5 7.73 mm to (195.7, 44.7), turned to 180 degrees
- moved Q1 4.02 mm to (207.8, 45.9)
- moved C13 1.51 mm to (207.0, 43.1)
- moved C5 0.72 mm to (238.8, 45.7)
- moved D6 0.50 mm to (238.1, 40.3)
- moved J3 0.49 mm to (192.1, 37.1)
- moved SW2 0.37 mm to (251.0, 40.9)
- moved BT2 0.34 mm to (222.9, 41.0)
- moved R5 0.18 mm to (233.4, 41.9)
- moved C8 0.07 mm to (233.4, 40.4)
- moved C6 0.05 mm to (241.8, 43.1)
- turned R11 to 0 degrees
Connections:
- J3 pad 1: +3V3 -> SCK
- J3 pad 10: GND -> +3V3
- J3 pad 2: CLK -> DRDY
- J3 pad 3: MOSI -> MISO
- J3 pad 4: MISO -> CS
- J3 pad 5: SCK -> MOSI
- J3 pad 6: DRDY -> GND
- J3 pad 7: CS -> CLK
- J4 pad 1: +3V3 -> SW_M
- J4 pad 10: GND -> DRDY_M
- J4 pad 2: CLK -> +3V3_M
- J4 pad 3: MOSI -> CLK_M
- J4 pad 4: MISO -> ADC_BAT_M
- J4 pad 5: SCK -> MOSI_M
- J4 pad 6: DRDY -> GND_M
- J4 pad 7: CS -> MISO_M
- J4 pad 8: ADC_BAT -> CS_M
- J4 pad 9: SW -> SCK_M
- U2 pad 3V3: +3V3 -> +3V3_M
- U2 pad GND: GND -> GND_M
- U2 pad P0.02: CLK -> CLK_M
- U2 pad P0.03: DRDY -> DRDY_M
- U2 pad P0.28: SW -> SW_M
- U2 pad P1.11: ADC_BAT -> ADC_BAT_M
- U2 pad P1.12: CS -> CS_M
- U2 pad P1.13: SCK -> SCK_M
- U2 pad P1.14: MISO -> MISO_M
- U2 pad P1.15: MOSI -> MOSI_M
Routing:
- net +3V3: track 0.00 -> 71.7 mm
- net ADC_BAT: track 0.00 -> 51.4 mm, vias 0 -> 1
- net GND: track 0.00 -> 40.5 mm, vias 0 -> 11
- net CS: track 0.00 -> 32.8 mm
- net CS_M: track 0.00 -> 31.8 mm
- net ADC_BAT_M: track 0.00 -> 31.8 mm
- net DRDY: track 0.00 -> 27.0 mm, vias 0 -> 1
- net SCK: track 0.00 -> 24.8 mm, vias 0 -> 1
- net MOSI: track 0.00 -> 24.7 mm, vias 0 -> 1
- net CLK: track 0.00 -> 24.5 mm, vias 0 -> 1
- net MISO: track 0.00 -> 23.8 mm, vias 0 -> 1
- net +VDD: track 0.00 -> 21.6 mm, vias 0 -> 1
- net SCK_M: track 0.00 -> 21.6 mm
- net GND_M: track 0.00 -> 20.0 mm, vias 0 -> 7
- net Net-(D6-K): track 0.00 -> 19.6 mm
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- added copper zone on B.Cu, net GND
- added copper zone on F.Cu, net GND
- added copper zone on B.Cu, net GND_M
- added copper zone on F.Cu, net GND_M
Other:
- board outline added: 91.9 x 55.4 mm
- board text removed: "20×32"
- board text removed: "72×15"

Commit message: Add files via upload
ガーバーファイル追加。
Parts:
- added ?: , , F.Cu at (248.7, 33.2)
- added ?: , , F.Cu at (249.6, 33.2)
- added REF**: MountingHole_2.1mm, MountingHole:MountingHole_2.1mm, F.Cu at (247.7, 33.2)
- moved U2 97.8 mm to (244.1, 11.5), turned to -90 degrees
- moved J4 76.3 mm to (239.4, 22.8), turned to 0 degrees
Other:
- board size 91.9 x 55.4 mm -> 72.1 x 47.9 mm
